File: Hardware/Magkeys.kicad_pcb (KiCad board)
At the start: 2 copper layers, 169 parts, among them SW1 SW_Push, SW10 SW_Push, SW11 SW_Push, SW12 SW_Push, SW13 SW_Push, SW14 SW_Push, SW15 SW_Push, SW16 SW_Push, SW17 SW_Push, SW18 SW_Push, SW19 SW_Push, SW2 SW_Push, SW20 SW_Push, SW21 SW_Push, SW22 SW_Push, SW23 SW_Push, SW24 SW_Push, SW25 SW_Push, SW26 SW_Push, SW27 SW_Push, SW28 SW_Push, SW29 SW_Push, SW3 SW_Push, SW30 SW_Push, SW31 SW_Push, SW32 SW_Push, SW33 SW_Push, SW34 SW_Push, SW35 SW_Push, SW36 SW_Push, SW37 SW_Push, SW38 SW_Push, SW39 SW_Push, SW4 SW_Push, SW40 SW_Push, SW41 SW_Push, SW42 SW_Push, SW43 SW_Push, SW44 SW_Push, SW45 SW_Push, SW46 SW_Push, SW47 SW_Push, SW48 SW_Push, SW49 SW_Push, SW5 SW_Push, SW50 SW_Push, SW51 SW_Push, SW52 SW_Push, SW53 SW_Push, SW54 SW_Push, SW55 SW_Push, SW56 SW_Push, SW57 SW_Push, SW58 SW_Push, SW59 SW_Push, SW6 SW_Push, SW60 SW_Push, SW61 SW_Push, SW62 SW_Push, SW63 SW_Push, SW64 SW_Push, SW65 SW_Push, SW66 SW_Push, SW67 SW_Push, SW68 SW_Push, SW69 SW_Push, SW7 SW_Push, SW70 SW_Push, SW71 SW_Push, SW72 SW_Push, SW73 SW_Push, SW74 SW_Push, SW75 SW_Push, SW76 SW_Push, SW77 SW_Push, SW78 SW_Push, SW79 SW_Push, SW8 SW_Push, SW80 SW_Push, SW81 SW_Push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

Commit message: did layout
Parts:
- A1: footprint Module:RaspberryPi_Pico_W_SMD_HandSolder -> Module:RaspberryPi_Pico_W_SMD
- moved D75 407.7 mm to (152.6, 253.0), turned to 90 degrees
- moved D1 405.9 mm to (150.2, 157.8), turned to 90 degrees
- moved D16 403.1 mm to (150.3, 176.8), turned to 90 degrees
- moved SW13 400.8 mm to (375.9, 156.2)
- moved SW19 400.8 mm to (185.4, 175.2)
- moved SW24 400.8 mm to (280.7, 175.2)
- moved SW29 400.8 mm to (375.9, 175.2)
- moved SW3 400.8 mm to (185.4, 156.2)
- moved SW41 400.8 mm to (328.3, 194.3)
- moved SW56 400.8 mm to (333.1, 213.3)
- moved SW62 400.8 mm to (190.2, 232.3)
- moved SW67 400.8 mm to (285.4, 232.3)
- moved SW79 400.8 mm to (337.8, 251.4)
- moved SW8 400.8 mm to (280.7, 156.2)
- moved SW1 400.8 mm to (147.3, 156.2)
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Connections:
- A1 pad 36: unconnected-(A1-3V3-Pad36) -> +3V3
- D21 pad 2: unconnected-(D21-A-Pad2) -> Net-(D21-A)
- D22 pad 2: unconnected-(D22-A-Pad2) -> Net-(D22-A)
- D25 pad 2: unconnected-(D25-A-Pad2) -> Net-(D25-A)
- D36 pad 2: unconnected-(D36-A-Pad2) -> Net-(D36-A)
- D37 pad 2: unconnected-(D37-A-Pad2) -> Net-(D37-A)
- D40 pad 2: unconnected-(D40-A-Pad2) -> Net-(D40-A)
- D5 pad 2: unconnected-(D5-A-Pad2) -> Net-(D5-A)
- D51 pad 2: unconnected-(D51-A-Pad2) -> Net-(D51-A)
- D52 pad 2: unconnected-(D52-A-Pad2) -> Net-(D52-A)
- D55 pad 2: unconnected-(D55-A-Pad2) -> Net-(D55-A)
- D6 pad 2: unconnected-(D6-A-Pad2) -> Net-(D6-A)
- D65 pad 2: unconnected-(D65-A-Pad2) -> Net-(D65-A)
- D66 pad 2: unconnected-(D66-A-Pad2) -> Net-(D66-A)
- D69 pad 2: unconnected-(D69-A-Pad2) -> Net-(D69-A)
- D79 pad 2: unconnected-(D79-A-Pad2) -> Net-(D79-A)
- D80 pad 2: unconnected-(D80-A-Pad2) -> Net-(D80-A)
- D83 pad 2: unconnected-(D83-A-Pad2) -> Net-(D83-A)
- D9 pad 2: unconnected-(D9-A-Pad2) -> Net-(D9-A)
- SW21 pad 1: unconnected-(SW21-Pad1) -> Net-(D21-A)
- SW22 pad 1: unconnected-(SW22-Pad1) -> Net-(D22-A)
- SW25 pad 1: unconnected-(SW25-Pad1) -> Net-(D25-A)
- SW36 pad 1: unconnected-(SW36-Pad1) -> Net-(D36-A)
- SW37 pad 1: unconnected-(SW37-Pad1) -> Net-(D37-A)
- SW40 pad 1: unconnected-(SW40-Pad1) -> Net-(D40-A)
- SW5 pad 1: unconnected-(SW5-Pad1) -> Net-(D5-A)
- SW51 pad 1: unconnected-(SW51-Pad1) -> Net-(D51-A)
- SW52 pad 1: unconnected-(SW52-Pad1) -> Net-(D52-A)
- SW55 pad 1: unconnected-(SW55-Pad1) -> Net-(D55-A)
- SW6 pad 1: unconnected-(SW6-Pad1) -> Net-(D6-A)
- SW65 pad 1: unconnected-(SW65-Pad1) -> Net-(D65-A)
- SW66 pad 1: unconnected-(SW66-Pad1) -> Net-(D66-A)
- SW69 pad 1: unconnected-(SW69-Pad1) -> Net-(D69-A)
- SW79 pad 1: unconnected-(SW79-Pad1) -> Net-(D79-A)
- SW80 pad 1: unconnected-(SW80-Pad1) -> Net-(D80-A)
- SW83 pad 1: unconnected-(SW83-Pad1) -> Net-(D83-A)
- SW9 pad 1: unconnected-(SW9-Pad1) -> Net-(D9-A)
Routing:
- net /COL6: track 0.00 -> 325.7 mm
- net /ROW8: track 0.00 -> 186.2 mm
- net /ROW10: track 0.00 -> 185.9 mm
- net /ROW9: track 0.00 -> 185.6 mm
- net /ROW7: track 0.00 -> 185.6 mm
- net /ROW4: track 0.00 -> 135.6 mm
- net /ROW2: track 0.00 -> 112.0 mm
- net /ROW3: track 0.00 -> 110.0 mm
- net /ROW1: track 0.00 -> 104.1 mm
- net /ROW5: track 0.00 -> 100.1 mm
- net /ROW6: track 0.00 -> 100.1 mm
- net /ROW14: track 0.00 -> 96.0 mm
- net /ROW13: track 0.00 -> 91.9 mm
- net /ROW12: track 0.00 -> 89.0 mm
- net /ROW11: track 0.00 -> 86.0 mm
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
Commit message: idk
Parts:
- moved A1 467.5 mm to (461.2, 179.0)
Connections:
- A1 pad 1: /ROW1 -> /ROW16
- A1 pad 10: /ROW8 -> /ROW9
- A1 pad 11: /ROW9 -> /ROW8
- A1 pad 12: /ROW10 -> /ROW7
- A1 pad 14: /ROW11 -> /ROW6
- A1 pad 15: /ROW12 -> /ROW5
- A1 pad 16: /ROW13 -> /ROW4
- A1 pad 17: /ROW14 -> /ROW3
- A1 pad 19: /ROW15 -> /ROW2
- A1 pad 2: /ROW2 -> /ROW15
- A1 pad 20: /ROW16 -> /ROW1
- A1 pad 21: /COL1 -> /COL6
- A1 pad 22: /COL2 -> /COL5
- A1 pad 24: /COL3 -> /COL4
- A1 pad 25: /COL4 -> /COL3
- A1 pad 26: /COL5 -> /COL2
- A1 pad 27: /COL6 -> /COL1
- A1 pad 4: /ROW3 -> /ROW14
- A1 pad 5: /ROW4 -> /ROW13
- A1 pad 6: /ROW5 -> /ROW12
- A1 pad 7: /ROW6 -> /ROW11
- A1 pad 9: /ROW7 -> /ROW10
Routing:
- net /COL1: track 0.00 -> 355.6 mm, vias 0 -> 16
- net /ROW16: track 0.00 -> 26.3 mm
- net GND: vias 0 -> 1
- added copper zone on B.Cu, net GND
- added copper zone on F.Cu, net GND
Other:
- board outline added: 338 x 114.6 mm

Commit message: Added numpad
Parts:
- added D100: 1N4148W, Diode_SMD:D_SOD-123, B.Cu at (76.1, 181.5)
- added D101: 1N4148W, Diode_SMD:D_SOD-123, B.Cu at (104.7, 181.5)
- added D85: 1N4148W, Diode_SMD:D_SOD-123, B.Cu at (66.6, 105.3)
- added D86: 1N4148W, Diode_SMD:D_SOD-123, B.Cu at (85.6, 105.3)
- added D87: 1N4148W, Diode_SMD:D_SOD-123, B.Cu at (104.7, 105.3)
- added D88: 1N4148W, Diode_SMD:D_SOD-123, B.Cu at (123.7, 105.3)
- added D89: 1N4148W, Diode_SMD:D_SOD-123, B.Cu at (66.6, 124.4)
- added D90: 1N4148W, Diode_SMD:D_SOD-123, B.Cu at (85.6, 124.4)
- added D91: 1N4148W, Diode_SMD:D_SOD-123, B.Cu at (104.7, 124.4)
- added D92: 1N4148W, Diode_SMD:D_SOD-123, B.Cu at (123.7, 133.9)
- added D93: 1N4148W, Diode_SMD:D_SOD-123, B.Cu at (66.6, 143.4)
- added D94: 1N4148W, Diode_SMD:D_SOD-123, B.Cu at (85.6, 143.4)
- added D95: 1N4148W, Diode_SMD:D_SOD-123, B.Cu at (104.7, 143.4)
- added D96: 1N4148W, Diode_SMD:D_SOD-123, B.Cu at (66.6, 162.5)
- added D97: 1N4148W, Diode_SMD:D_SOD-123, B.Cu at (85.6, 162.5)
- added D98: 1N4148W, Diode_SMD:D_SOD-123, B.Cu at (104.7, 162.5)
- added D99: 1N4148W, Diode_SMD:D_SOD-123, B.Cu at (123.7, 172.0)
- added SW100: SW_Push, Button_Switch_Keyboard:SW_Cherry_MX_2.00u_Plate, F.Cu at (73.2, 179.9)
- added SW101: SW_Push, Button_Switch_Keyboard:SW_Cherry_MX_1.00u_Plate, F.Cu at (101.8, 179.9)
- added SW85: SW_Push, Button_Switch_Keyboard:SW_Cherry_MX_1.00u_Plate, F.Cu at (63.6, 103.7)
- added SW86: SW_Push, Button_Switch_Keyboard:SW_Cherry_MX_1.00u_Plate, F.Cu at (82.7, 103.7)
- added SW87: SW_Push, Button_Switch_Keyboard:SW_Cherry_MX_1.00u_Plate, F.Cu at (101.8, 103.7)
- added SW88: SW_Push, Button_Switch_Keyboard:SW_Cherry_MX_1.00u_Plate, F.Cu at (120.8, 103.7)
- added SW89: SW_Push, Button_Switch_Keyboard:SW_Cherry_MX_1.00u_Plate, F.Cu at (63.6, 122.7)
- added SW90: SW_Push, Button_Switch_Keyboard:SW_Cherry_MX_1.00u_Plate, F.Cu at (82.7, 122.7)
- added SW91: SW_Push, Button_Switch_Keyboard:SW_Cherry_MX_1.00u_Plate, F.Cu at (101.8, 122.7)
- added SW92: SW_Push, Button_Switch_Keyboard:SW_Cherry_MX_2.00u_Vertical_Plate, F.Cu at (120.8, 132.2)
- added SW93: SW_Push, Button_Switch_Keyboard:SW_Cherry_MX_1.00u_Plate, F.Cu at (63.6, 141.8)
- added SW94: SW_Push, Button_Switch_Keyboard:SW_Cherry_MX_1.00u_Plate, F.Cu at (82.7, 141.8)
- added SW95: SW_Push, Button_Switch_Keyboard:SW_Cherry_MX_1.00u_Plate, F.Cu at (101.8, 141.8)
- added SW96: SW_Push, Button_Switch_Keyboard:SW_Cherry_MX_1.00u_Plate, F.Cu at (63.6, 160.8)
- added SW97: SW_Push, Button_Switch_Keyboard:SW_Cherry_MX_1.00u_Plate, F.Cu at (82.7, 160.8)
- added SW98: SW_Push, Button_Switch_Keyboard:SW_Cherry_MX_1.00u_Plate, F.Cu at (101.8, 160.8)
- added SW99: SW_Push, Button_Switch_Keyboard:SW_Cherry_MX_2.00u_Vertical_Plate, F.Cu at (120.8, 170.3)
- moved D21 35.3 mm to (261.8, 176.8)
- moved D22 35.3 mm to (280.7, 176.8)
- moved D37 35.3 mm to (290.4, 195.8)
- moved D6 35.3 mm to (281.1, 157.7)
- moved SW22 35.3 mm to (277.9, 175.1)
- moved SW6 35.3 mm to (277.9, 156.1)
- moved SW65 35.3 mm to (282.6, 232.3)
- moved A1 35.3 mm to (496.4, 178.9)
- moved D1 35.3 mm to (185.5, 157.7)
- moved D10 35.3 mm to (357.2, 157.7)
- moved D11 35.3 mm to (376.0, 157.7)
- moved D12 35.3 mm to (395.3, 157.7)
- moved D13 35.3 mm to (414.4, 157.7)
- moved D14 35.3 mm to (433.4, 157.7)
- moved D15 35.3 mm to (452.3, 157.7)
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Routing:
- net /COL5: track 0.00 -> 421.9 mm, vias 0 -> 15
- net /COL4: track 0.00 -> 404.3 mm, vias 0 -> 15
- net /COL2: track 0.00 -> 400.2 mm, vias 0 -> 16
- net /COL3: track 0.00 -> 392.1 mm, vias 0 -> 16
- net /ROW1: track 104.1 -> 422.3 mm
- net /ROW5: track 100.1 -> 417.5 mm, vias 0 -> 1
- net /ROW6: track 100.1 -> 398.6 mm, vias 0 -> 2
- net /ROW2: track 112.0 -> 395.9 mm, vias 0 -> 1
- net /ROW3: track 110.0 -> 376.7 mm
- net /ROW4: track 135.6 -> 386.4 mm, vias 0 -> 1
- net /ROW7: track 185.6 -> 382.4 mm, vias 0 -> 1
- net /ROW8: track 186.2 -> 365.2 mm, vias 0 -> 1
- net /ROW9: track 185.6 -> 347.2 mm, vias 0 -> 1
- net /ROW10: track 185.9 -> 329.7 mm, vias 0 -> 1
- net /ROW11: track 86.0 -> 214.7 mm, vias 0 -> 1
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
Commit message: Completed PCB
Parts:
- added REF**: MouseBite-Slot_2.0x2.0mm_outset_D0.5mm_P0.85mm_3h, Panelization:MouseBite-Slot_2.0x2.0mm_outset_D0.5mm_P0.85mm_3h, F.Cu at (170.4, 215.1)
- added REF**: MouseBite-Slot_2.0x2.0mm_outset_D0.5mm_P0.85mm_3h, Panelization:MouseBite-Slot_2.0x2.0mm_outset_D0.5mm_P0.85mm_3h, F.Cu at (170.4, 253.7)
- added REF**: MouseBite-Slot_2.0x2.0mm_outset_D0.5mm_P0.85mm_3h, Panelization:MouseBite-Slot_2.0x2.0mm_outset_D0.5mm_P0.85mm_3h, F.Cu at (170.4, 185.1)
- added U1: Seeeduino Xiao rp2040, PCM_marbastlib-xp-promicroish:Xiao_rp2040_AC_Reflow, F.Cu at (84.9, 182.7)
- moved D88 82.1 mm to (164.2, 176.8)
- moved D90 82.1 mm to (126.1, 195.8)
- moved D92 82.1 mm to (164.2, 205.4)
- moved SW85 82.1 mm to (104.1, 175.1)
- moved SW88 82.1 mm to (161.3, 175.1)
- moved SW89 82.1 mm to (104.1, 194.2)
- moved SW90 82.1 mm to (123.2, 194.2)
- moved SW91 82.1 mm to (142.2, 194.2)
- moved SW92 82.1 mm to (161.3, 203.7)
- moved SW93 82.1 mm to (104.1, 213.2)
- moved SW96 82.1 mm to (104.1, 232.3)
- moved SW99 82.1 mm to (161.3, 241.8)
- moved D100 82.1 mm to (116.6, 253.0)
- moved D101 82.1 mm to (145.1, 253.0)
- moved D85 82.1 mm to (107.0, 176.8)
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Routing:
- net /NUM_ROW5: track 32.0 -> 122.9 mm, vias 0 -> 1
- net /NUM_ROW4: track 72.8 -> 142.7 mm
- net /NUM_COL4: track 66.7 -> 134.4 mm
- net /NUM_ROW3: track 49.1 -> 100.8 mm
- net /NUM_COL3: track 57.1 -> 105.1 mm
- net /NUM_ROW2: track 73.4 -> 114.7 mm, vias 4 -> 5
- net /NUM_ROW1: track 73.2 -> 106.7 mm, vias 4 -> 5
- net /NUM_COL2: track 86.7 -> 114.6 mm, vias 0 -> 1
- net /NUM_COL1: track 80.1 -> 87.8 mm
- net Net-(D99-A): track 0.00 -> 2.91 mm
- net Net-(D92-A): track 0.00 -> 2.91 mm
- net GND: vias 2 -> 4
Other:
- board size 338 x 114.6 mm -> 434.9 x 114.6 mm

Commit message: changes in the PCB
Parts:
- added J1: Conn_01x04_Pin, Connector_PinHeader_2.54mm:PinHeader_1x04_P2.54mm_Vertical, F.Cu at (502.2, 216.5)
- added SW102: RotaryEncoder, Rotary_Encoder:RotaryEncoder_Alps_EC11E_Vertical_H20mm, F.Cu at (495.5, 235.5)
- SW1, SW10, SW101, SW11, SW12, SW13, SW14, SW15, SW16, SW17, SW18, SW19, SW2, SW20, SW21, SW22, SW23, SW24, SW25, SW26, SW27, SW28, SW29, SW3, SW31, SW33, SW34, SW35, SW36, SW37, SW38, SW39, SW4, SW40, SW41, SW42, SW43, SW44, SW46, SW48, SW49, SW5, SW50, SW51, SW52, SW53, SW54, SW55, SW56, SW57, SW58, SW6, SW60, SW62, SW63, SW64, SW65, SW66, SW67, SW68, SW69, SW7, SW70, SW71, SW73, SW74, SW79, SW8, SW80, SW81, SW82, SW83, SW84, SW85, SW86, SW87, SW88, SW89, SW9, SW90, SW91, SW93, SW94, SW95, SW96, SW97, SW98: footprint Button_Switch_Keyboard:SW_Cherry_MX_1.00u_Plate -> easyeda2kicad:SW_Cherry_MX_1.00u_Plate
- SW100, SW30: footprint Button_Switch_Keyboard:SW_Cherry_MX_2.00u_Plate -> easyeda2kicad:SW_Cherry_MX_2.00u_Plate
- SW32, SW45: footprint Button_Switch_Keyboard:SW_Cherry_MX_1.50u_Plate -> easyeda2kicad:SW_Cherry_MX_1.50u_Plate
- SW47, SW72: footprint Button_Switch_Keyboard:SW_Cherry_MX_1.75u_Plate -> easyeda2kicad:SW_Cherry_MX_1.75u_Plate
- SW59, SW61: footprint Button_Switch_Keyboard:SW_Cherry_MX_2.25u_Plate -> easyeda2kicad:SW_Cherry_MX_2.25u_Plate
- SW75, SW76, SW77: footprint Button_Switch_Keyboard:SW_Cherry_MX_1.25u_Plate -> easyeda2kicad:SW_Cherry_MX_1.25u_Plate
- SW78: footprint Button_Switch_Keyboard:SW_Cherry_MX_6.25u_Plate -> easyeda2kicad:SW_Cherry_MX_6.25u_Plate
- SW92, SW99: footprint Button_Switch_Keyboard:SW_Cherry_MX_2.00u_Vertical_Plate -> easyeda2kicad:SW_Cherry_MX_2.00u_Vertical_Plate
Connections:
- A1 pad 21: /COL6 -> /U0_TX
- A1 pad 22: /COL5 -> /U0_RX
- A1 pad 24: /COL4 -> /COL6
- A1 pad 25: /COL3 -> /COL5
- A1 pad 26: /COL2 -> /COL4
- A1 pad 27: /COL1 -> /COL3
- A1 pad 29: unconnected-(A1-GPIO22-Pad29) -> /COL2
- A1 pad 31: unconnected-(A1-GPIO26_ADC0-Pad31) -> /COL1
- A1 pad 32: unconnected-(A1-GPIO27_ADC1-Pad32) -> /ENC_A
- A1 pad 34: unconnected-(A1-GPIO28_ADC2-Pad34) -> /ENC_B
Routing:
- net VBUS: track 0.00 -> 113.4 mm, vias 0 -> 2
- net /ENC_A: track 0.00 -> 93.4 mm, vias 0 -> 2
- net /ENC_B: track 0.00 -> 92.4 mm, vias 0 -> 2
- net /U0_RX: track 0.00 -> 86.1 mm, vias 0 -> 1
- net /U0_TX: track 0.00 -> 86.1 mm, vias 0 -> 1
- net /COL2: track 400.2 -> 423.1 mm, vias 16 -> 15
- net /COL6: track 425.5 -> 420.0 mm
- net /COL1: track 402.1 -> 397.6 mm
- net /COL5: track 421.9 -> 418.3 mm
- net GND: track 0.00 -> 3.16 mm, vias 4 -> 13
- net /COL3: track 392.1 -> 393.9 mm, vias 16 -> 15
- net /ROW1: track 422.3 -> 423.8 mm
- net /ROW14: track 162.8 -> 162.0 mm
- net /ROW13: track 185.1 -> 185.8 mm
- net /COL4: track 404.3 -> 404.7 mm, vias 15 -> 14
Other:
- outline, holes or cut-outs redrawn
