File: Hardware/Magkeys.kicad_pcb (KiCad board)
At the start: 2 copper layers, 434.9 x 114.6 mm, 209 parts, among them J1 Conn_01x04_Pin, SW1 SW_Push, SW10 SW_Push, SW100 SW_Push, SW101 SW_Push, SW102 RotaryEncoder, SW11 SW_Push, SW12 SW_Push, SW13 SW_Push, SW14 SW_Push, SW15 SW_Push, SW16 SW_Push, SW17 SW_Push, SW18 SW_Push, SW19 SW_Push, SW2 SW_Push, SW20 SW_Push, SW21 SW_Push, SW22 SW_Push, SW23 SW_Push, SW24 SW_Push, SW25 SW_Push, SW26 SW_Push, SW27 SW_Push, SW28 SW_Push, SW29 SW_Push, SW3 SW_Push, SW30 SW_Push, SW31 SW_Push, SW32 SW_Push, SW33 SW_Push, SW34 SW_Push, SW35 SW_Push, SW36 SW_Push, SW37 SW_Push, SW38 SW_Push, SW39 SW_Push, SW4 SW_Push, SW40 SW_Push, SW41 SW_Push, SW42 SW_Push, SW43 SW_Push, SW44 SW_Push, SW45 SW_Push, SW46 SW_Push, SW47 SW_Push, SW48 SW_Push, SW49 SW_Push, SW5 SW_Push, SW50 SW_Push, SW51 SW_Push, SW52 SW_Push, SW53 SW_Push, SW54 SW_Push, SW55 SW_Push, SW56 SW_Push, SW57 SW_Push, SW58 SW_Push, SW59 SW_Push, SW6 SW_Push, SW60 SW_Push, SW61 SW_Push, SW62 SW_Push, SW63 SW_Push, SW64 SW_Push, SW65 SW_Push, SW66 SW_Push, SW67 SW_Push, SW68 SW_Push, SW69 SW_Push, SW7 SW_Push, SW70 SW_Push, SW71 SW_Push, SW72 SW_Push, SW73 SW_Push, SW74 SW_Push, SW75 SW_Push, SW76 SW_Push, SW77 SW_Push, SW78 SW_Push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

Commit message: 3d files generated, PCB updated and production files generated too
Parts:
- removed SW102: RotaryEncoder, Rotary_Encoder:RotaryEncoder_Alps_EC11E_Vertical_H20mm
- added C1: 15p, Capacitor_SMD:C_0402_1005Metric, F.Cu at (85.3, 242.0)
- added C10: 1u, Capacitor_SMD:C_0402_1005Metric, F.Cu at (94.7, 253.9)
- added C11: 100n, Capacitor_SMD:C_0402_1005Metric, F.Cu at (84.2, 256.9)
- added C12: 100n, Capacitor_SMD:C_0402_1005Metric, F.Cu at (85.2, 245.0)
- added C13: 100n, Capacitor_SMD:C_0402_1005Metric, F.Cu at (83.2, 256.9)
- added C14: 10u, Capacitor_SMD:C_0402_1005Metric, F.Cu at (78.9, 239.2)
- added C15: 10u, Capacitor_SMD:C_0402_1005Metric, F.Cu at (84.3, 242.9)
- added C2: 15p, Capacitor_SMD:C_0402_1005Metric, F.Cu at (88.9, 244.1)
- added C3: 100n, Capacitor_SMD:C_0402_1005Metric, F.Cu at (87.2, 255.2)
- added C4: 100n, Capacitor_SMD:C_0402_1005Metric, F.Cu at (86.0, 244.1)
- added C5: 100n, Capacitor_SMD:C_0402_1005Metric, F.Cu at (94.7, 252.9)
- added C6: 100n, Capacitor_SMD:C_0402_1005Metric, F.Cu at (84.2, 255.1)
- added C7: 100n, Capacitor_SMD:C_0402_1005Metric, F.Cu at (83.3, 255.1)
- added C8: 100n, Capacitor_SMD:C_0402_1005Metric, F.Cu at (89.0, 263.3)
- added C9: 100n, Capacitor_SMD:C_0402_1005Metric, F.Cu at (92.8, 248.7)
- added H1: MountingHole, MountingHole:MountingHole_3.2mm_M3, B.Cu at (418.2, 170.7)
- added H2: MountingHole, MountingHole:MountingHole_3.2mm_M3, B.Cu at (456.3, 227.9)
- added H3: MountingHole, MountingHole:MountingHole_3.2mm_M3, B.Cu at (160.0, 189.9)
- added H4: MountingHole, MountingHole:MountingHole_3.2mm_M3, B.Cu at (158.9, 258.8)
- added H5: MountingHole, MountingHole:MountingHole_3.2mm_M3, B.Cu at (111.1, 189.8)
- added H6: MountingHole, MountingHole:MountingHole_3.2mm_M3, B.Cu at (65.7, 261.6)
- added H7: MountingHole, MountingHole:MountingHole_3.2mm_M3, B.Cu at (203.9, 227.8)
- added H8: MountingHole, MountingHole:MountingHole_3.2mm_M3, B.Cu at (208.6, 170.7)
- added J2: USB_C_Receptacle_USB2.0_16P, Connector_USB:USB_C_Receptacle_XKB_U262-16XN-4BVC11, F.Cu at (64.1, 242.1)
- added J3: Conn_01x04_Pin, Connector_PinHeader_2.54mm:PinHeader_1x04_P2.54mm_Vertical, F.Cu at (82.1, 236.9)
- added JP1: Jumper_2_Open, Jumper:SolderJumper-2_P1.3mm_Open_TrianglePad1.0x1.5mm, F.Cu at (82.1, 244.8)
- added L1: 1u, Inductor_SMD:L_0402_1005Metric, F.Cu at (84.8, 240.1)
- added R1: 10k, Resistor_SMD:R_0402_1005Metric, F.Cu at (82.8, 243.0)
- added R2: 5.1k, Resistor_SMD:R_0402_1005Metric, F.Cu at (70.4, 240.9)
- added R3: 5.1k, Resistor_SMD:R_0402_1005Metric, F.Cu at (70.6, 243.8)
- added R4: 27, Resistor_SMD:R_0402_1005Metric, F.Cu at (86.0, 258.0)
- added R5: 27, Resistor_SMD:R_0402_1005Metric, F.Cu at (85.1, 258.0)
- added R6: 1k, Resistor_SMD:R_0402_1005Metric, F.Cu at (87.5, 244.5)
- added R7: 10k, Resistor_SMD:R_0402_1005Metric, F.Cu at (96.4, 258.5)
- added SW103: RotaryEncoder_Switch_MP, Rotary_Encoder:RotaryEncoder_Alps_EC11E-Switch_Vertical_H20mm_MountingHoles, F.Cu at (78.2, 248.9)
- added SW104: SW_Push, Button_Switch_SMD:SW_SPST_PTS810, F.Cu at (85.4, 262.7)
- added U2: RP2040, Package_DFN_QFN:QFN-56-1EP_7x7mm_P0.4mm_EP3.2x3.2mm, F.Cu at (87.4, 250.0)
- added U3: ADP2108AUJ-3.3, Package_TO_SOT_SMD:TSOT-23-5, F.Cu at (82.2, 240.5)
- added Y1: 12 MHz, Crystal:Crystal_SMD_3225-4Pin_3.2x2.5mm, F.Cu at (87.8, 241.8)
- U1: value Seeeduino Xiao rp2040 -> W25Q128JVP; footprint PCM_marbastlib-xp-promicroish:Xiao_rp2040_AC_Reflow -> Package_SON:WSON-8-1EP_6x5mm_P1.27mm_EP3.4x4.3mm
- moved U1 77.5 mm to (91.2, 259.9), turned to 180 degrees
- moved J1 13.5 mm to (488.8, 216.9), turned to 90 degrees
Connections:
- A1 pad 32: /ENC_A -> unconnected-(A1-GPIO27_ADC1-Pad32)
- A1 pad 34: /ENC_B -> unconnected-(A1-GPIO28_ADC2-Pad34)
- U1 pad 1: unconnected-(U1-P26-Pad1) -> /QSPI_CS
- U1 pad 2: unconnected-(U1-P27-Pad2) -> /QSPI_IO1
- U1 pad 3: /NUM_ROW1 -> /QSPI_IO2
- U1 pad 4: /NUM_ROW2 -> GND
- U1 pad 5: /NUM_ROW3 -> /QSPI_IO0
- U1 pad 6: /NUM_ROW4 -> /QSPI_CLK
- U1 pad 7: /NUM_ROW5 -> /QSPI_IO3
- U1 pad 8: +5V -> +3V3
Routing:
- net /ENC_A: track 93.4 -> 6.70 mm, vias 2 -> 0
- net /ENC_B: track 92.4 -> 11.9 mm, vias 2 -> 0
- net +3V3: track 0.00 -> 70.2 mm, vias 0 -> 4
- net /NUM_ROW5: track 122.9 -> 63.7 mm
- net /NUM_ROW4: track 142.7 -> 94.6 mm
- net /NUM_ROW1: track 106.7 -> 147.6 mm, vias 5 -> 4
- net /USB_DP: track 0.00 -> 40.5 mm, vias 0 -> 2
- net /USB_DN: track 0.00 -> 40.0 mm, vias 0 -> 2
- net /QSPI_CS: track 0.00 -> 25.8 mm
- net GND: track 3.16 -> 24.8 mm, vias 13 -> 43
- net /ENC_S1: track 0.00 -> 18.5 mm
- net +1V1: track 0.00 -> 17.9 mm, vias 0 -> 2
- net /NUM_COL2: track 114.6 -> 131.2 mm, vias 1 -> 0
- net /ENC_S2: track 0.00 -> 16.0 mm
- net /U00_RX: track 0.00 -> 15.8 mm
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Other:
- board size 434.9 x 114.6 mm -> 447 x 114.6 mm
